File: vWAN-macropad/vWAN-macropad.kicad_pcb (KiCad board)
At the start: 2 copper layers, 92.7 x 59.8 mm, 18 parts, among them J1 OLED_128x32, SW1 Switch, SW2 Switch, SW3 Switch, SW4 Switch, SW5 Switch, SW6 Switch, SW7 RotaryEncoder_Switch, U1 YAAJ_WeAct_BlackPill_Part_Lik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

Commit message: Update preliminary trace arrangement
Connections:
- D7 pad 1: Row 0 -> ENC_SW2
- SW7 pad S1: Col 3 -> ENC_SW1
- U1 pad 1: ENC_A -> ENC_B
- U1 pad 10: Row 0 -> ENC_SW2
- U1 pad 11: unconnected-(U1-PB3-Pad11) -> Row 0
- U1 pad 2: ENC_B -> ENC_A
- U1 pad 4: unconnected-(U1-PB15-Pad4) -> ENC_SW1
- U1 pad 5: Col 3 -> unconnected-(U1-PA8-Pad5)
Routing:
- net +3.3V: track 0.00 -> 171.5 mm, vias 0 -> 1
- net GND: track 0.00 -> 148.4 mm
- net SDA: track 0.00 -> 87.2 mm, vias 0 -> 2
- net SCL-SCK: track 0.00 -> 83.9 mm, vias 0 -> 2
- net ENC_B: track 0.00 -> 39.7 mm
- net ENC_A: track 0.00 -> 33.5 mm
- net ENC_SW2: track 0.00 -> 18.5 mm
- net ENC_SW1: track 0.00 -> 12.2 mm
- net Net-(D7-A): track 0.00 -> 3.73 mm
- net Row 0: track 52.1 -> 49.5 mm
- net Col 1: track 89.2 -> 89.7 mm

Commit message: Edit near final schematic + PCB
Parts:
- added H1: MountingHole_Pad, MountingHole:MountingHole_2.2mm_M2_DIN965, F.Cu at (125.4, 78.4)
- added H2: MountingHole_Pad, MountingHole:MountingHole_2.2mm_M2_DIN965, F.Cu at (220.3, 78.4)
- added H3: MountingHole_Pad, MountingHole:MountingHole_2.2mm_M2_DIN965, F.Cu at (125.4, 135.6)
- added H4: MountingHole_Pad, MountingHole:MountingHole_2.2mm_M2_DIN965, F.Cu at (220.3, 135.6)
Routing:
- net GND: track 148.4 -> 0.03 mm
- net Col 0: track 108.2 -> 114.0 mm
- net ENC_B: track 39.7 -> 44.6 mm
- net +3.3V: track 171.5 -> 174.8 mm
- net Col 1: track 89.7 -> 91.2 mm
- net Col 2: track 49.1 -> 50.0 mm
- added copper zone on B.Cu, net GND
- added copper zone on F.Cu, net GND
Other:
- board size 92.7 x 59.8 mm -> 100.8 x 63.1 mm
- board text added: "microWAN | Designed by wandou"
- board text added: "v1.0"

Commit message: Add files via upload
Parts:
- added C3: 2.2uF, Capacitor_THT:C_Disc_D7.5mm_W4.4mm_P5.00mm, F.Cu at (189.4, 120.1)
- added C4: 2.2uF, Capacitor_THT:C_Disc_D7.5mm_W4.4mm_P5.00mm, F.Cu at (217.8, 90.3)
- H1, H2, H3, H4: footprint MountingHole:MountingHole_2.2mm_M2_DIN965 -> MountingHole:MountingHole_2.2mm_M2_ISO7380
- SW1, SW2, SW3, SW4, SW5, SW6: moved to B.Cu
- moved J1 39.8 mm to (167.1, 94.9), turned to 180 degrees
- moved D2 19.1 mm to (148.1, 112.8)
- moved D5 19.1 mm to (148.1, 131.8)
- moved D1 19.0 mm to (129.0, 112.8)
- moved D3 19.0 mm to (167.1, 112.8)
- moved D4 19.0 mm to (129.0, 131.8)
- moved D6 19.0 mm to (167.1, 131.8)
- moved C2 12.0 mm to (189.4, 130.1)
- moved D7 1.27 mm to (187.5, 93.7)
- moved C1 0.77 mm to (216.8, 84.7)
- moved U1 0.77 mm to (196.1, 82.2)
- moved SW7 0.41 mm to (176.7, 87.6)
- turned SW1 to 180 degrees
- turned SW2 to 180 degrees
- turned SW3 to 180 degrees
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Connections:
- D1 pad 1: Row 0 -> Row 1
- D2 pad 1: Row 0 -> Row 1
- D3 pad 1: Row 0 -> Row 1
- D4 pad 1: Row 1 -> Row 2
- D5 pad 1: Row 1 -> Row 2
- D6 pad 1: Row 1 -> Row 2
- D7 pad 1: ENC_SW2 -> Row 0
- SW7 pad S1: ENC_SW1 -> Col 2
- U1 pad 10: ENC_SW2 -> Row 1
- U1 pad 11: Row 0 -> unconnected-(U1-PB3-Pad11)
- U1 pad 12: Col 2 -> Row 2
- U1 pad 27: Row 1 -> unconnected-(U1-PA1-Pad27)
- U1 pad 4: ENC_SW1 -> Col 2
- U1 pad 5: unconnected-(U1-PA8-Pad5) -> Row 0
Routing:
- net Row 2: track 0.00 -> 81.2 mm
- net Row 0: track 49.5 -> 9.21 mm
- net SDA: track 87.2 -> 48.8 mm
- net SCL-SCK: track 83.9 -> 48.4 mm
- net Col 0: track 114.0 -> 92.5 mm
- net ENC_SW2: track 18.5 -> 0.00 mm
- net +3.3V: track 174.8 -> 157.9 mm, vias 1 -> 2
- net Col 1: track 91.2 -> 74.8 mm
- net Row 1: track 84.1 -> 70.3 mm
- net ENC_SW1: track 12.2 -> 0.00 mm
- net Col 2: track 50.0 -> 45.3 mm
- net ENC_B: track 44.6 -> 42.7 mm
Other:
- board text added: "SEP/17/2025 - v1.0"
- board text added: "macroWAN | Designed by wandou"
- board text removed: "microWAN | Designed by wandou"
- board text removed: "v1.0"
