File: vWAN-macropad/vWAN-macropad.kicad_sch (KiCad schematic)
At the start: 0 parts

Commit message: Add Blackpill v3.1 schematic
Parts:
- added D1, D2, D3, D4, D5, D6: Diode, symbol ScottoKeebs:Placeholder_Diode
- added SW1, SW2, SW3, SW4, SW5, SW6: Switch, symbol ScottoKeebs:Placeholder_Switch
Connections:
- new net: D1.1 (K), D2.1 (K), D3.1 (K)
- new net: D2.2 (A), SW2.2
- new net: SW2.1, SW5.1
- new net: D4.1 (K), D5.1 (K), D6.1 (K)
- new net: D5.2 (A), SW5.2
- new net: SW1.1, SW4.1
- new net: D1.2 (A), SW1.2
- new net: D4.2 (A), SW4.2
- new net: D6.2 (A), SW6.2
- new net: SW3.1, SW6.1
- new net: D3.2 (A), SW3.2
Other:
- company: (none) -> Author: Brendan Leung
- title: (none) -> vWAN macropad

Commit message: Add submodules and edit schematics
Parts:
- added D7: Diode, symbol ScottoKeebs:Placeholder_Diode
- added J1: OLED_128x32, ScottoKeebs_Components:OLED_128x32, symbol ScottoKeebs:OLED_128x32
- added SW7: RotaryEncoder_Switch, symbol Device:RotaryEncoder_Switch
- added U1: ~, symbol Blackpill_v3.1:Blackpill_Dev_Board
Connections:
- net Row 0: now reaches D1.1 (K), D2.1 (K), D3.1 (K)
- net Row 0: now also D7.1 (K)
- net at D2.2 (A): now also SW2.1; no longer SW2.2
- net at SW5.1: now also D5.2 (A); no longer SW2.1
- net Row 1: now reaches D4.1 (K), D5.1 (K), D6.1 (K)
- net Col 1: now reaches SW5.2
- net Col 1: now also SW2.2; no longer D5.2 (A)
- net at SW1.1: now also D1.2 (A); no longer SW4.1
- net Col 0: now reaches SW1.2
- net Col 0: now also SW4.2; no longer D1.2 (A)
- net at D4.2 (A): now also SW4.1; no longer SW4.2
- net at D6.2 (A): now also SW6.1; no longer SW6.2
- net at SW3.1: now also D3.2 (A); no longer SW6.1
- net Col 2: now reaches SW3.2
- net Col 2: now also SW6.2; no longer D3.2 (A)
- new net: D7.2 (A), SW7.S2
- new net +3.3V: U1.20 (VB), U1.3 (3.3V)
- new net +5V: U1.1 (5V), U1.18 (PC14)
- new net Col 3: SW7.S1
- new net ENC_A: SW7.A
- new net ENC_B: SW7.B
- new net GND: J1.1 (GND), SW7.C, U1.19 (PC13), U1.2 (GND)
- new net SCL-SCK: J1.3 (SCL)
- new net SDA: J1.4 (SDA)
- new net VCC: J1.2 (VCC)
Other:
- moved on the sheet: D1, D2, D3, SW1, SW2, SW3

Commit message: Update schematic + PCB files
Parts:
- removed U1: ~, symbol Blackpill_v3.1:Blackpill_Dev_Board
- added C1, C2: 0.1uF, Capacitor_THT:C_Disc_D5.0mm_W2.5mm_P2.50mm, symbol Device:C
- added U1: YAAJ_WeAct_BlackPill_Part_Like_SWD_Breakout, Footprints:YAAJ_WeAct_BlackPill_SWD_2, symbol YAAJ_WeAct_BlackPill_Part_Like_SWD_Breakout:YAAJ_WeAct_BlackPill_Part_Like_SWD_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
- D1, D2, D3, D4, D5, D6, D7: footprint (none) -> ScottoKeebs_Components:Diode_DO-35
- SW1, SW2, SW3, SW4, SW5, SW6: footprint (none) -> MX_Hotswap:MX-Hotswap-1U
- SW7: footprint (none) -> Keebio-Parts:RotaryEncoder_EC11
Connections:
- net VCC is gone; now on net +3.3V: J1.2 (VCC)
- net +3.3V: now also C1.2, C2.2, U1.20 (3V3), U1.38 (3V3)
- net Col 0: now also U1.17 (PB9)
- net Col 1: now also U1.16 (PB8)
- net Col 2: now also U1.12 (PB4)
- net Col 3: now also U1.5 (PA8)
- net ENC_A: now also U1.1 (PB12)
- net ENC_B: now also U1.2 (PB13)
- net GND: now also C1.1, C2.1, U1.19 (GND), U1.39 (GND)
- net Row 0: now also U1.10 (PA15)
- net Row 1: now also U1.27 (PA1)
- net SCL-SCK: now also U1.14 (PB6)
- net SDA: now also U1.15 (PB7)
- no-connect marks 0 -> 22
Other:
- company: Author: Brendan Leung -> Author: wandou
- moved on the sheet: D1, D2, D3, D4, D5, D6, D7, J1, SW1, SW2, SW3, SW4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

Commit message: Edit project files
Connections:
- net ENC_A: now also U1.2 (PB13); no longer U1.1 (PB12)
- net ENC_B: now also U1.1 (PB12); no longer U1.2 (PB13)
- net Row 0: now also U1.11 (PB3); no longer D7.1 (K), U1.10 (PA15)
- net ENC_SW1: now reaches U1.4 (PB15)
- net ENC_SW1: now also SW7.S1
- net Col 3: no longer names the net of U1.5 (PA8)
- net Col 3: no longer SW7.S1
- new net ENC_SW2: D7.1 (K), U1.10 (PA15)
- no-connect marks 22 -> 29
Other:
- moved on the sheet: D7

Commit message: Edit near final schematic + PCB
Parts:
- added H1, H2, H3, H4: MountingHole_Pad, MountingHole:MountingHole_2.2mm_M2_DIN965, symbol Mechanical:MountingHole_Pad
Connections:
- net GND: now also H1.1, H2.1, H3.1, H4.1
Other:
- moved on the sheet: C1, C2, D7, SW7, U1

Commit message: Add files via upload
Parts:
- added C3, C4: 2.2uF, Capacitor_THT:C_Disc_D7.5mm_W4.4mm_P5.00mm, symbol Device:C
- H1, H2, H3, H4: footprint MountingHole:MountingHole_2.2mm_M2_DIN965 -> MountingHole:MountingHole_2.2mm_M2_ISO7380
Connections:
- net ENC_SW1 is gone; now on net Col 2: SW7.S1, U1.4 (PB15)
- net +3.3V: now also C3.2, C4.2
- net Col 2: no longer U1.12 (PB4)
- net GND: now also C3.1, C4.1
- net Row 0: now also D7.1 (K), U1.5 (PA8); no longer D1.1 (K), D2.1 (K), D3.1 (K), U1.11 (PB3)
- net Row 1: now also D1.1 (K), D2.1 (K), D3.1 (K), U1.10 (PA15); no longer D4.1 (K), D5.1 (K), D6.1 (K), U1.27 (PA1)
- removed net ENC_SW2: D7.1 (K), U1.10 (PA15)
- new net Row 2: D4.1 (K), D5.1 (K), D6.1 (K), U1.12 (PB4)
- no-connect marks 29 -> 30
Other:
- company: Author: wandou -> (none)
- title: vWAN macropad -> microWAN
- moved on the sheet: D7, H1, H2, H3, H4, J1, SW7
