File: macroWAN/vWAN-macropad.kicad_pcb (KiCad board)
At the start: 2 copper layers, 100.8 x 63.1 mm, 24 parts, among them J1 OLED_128x32, SW1 Switch, SW2 Switch, SW3 Switch, SW4 Switch, SW5 Switch, SW6 Switch, SW7 RotaryEncoder_Switch, U1 YAAJ_WeAct_BlackPill_Part_Lik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

Commit message: Add finalized firmware
Routing:
- net Col 2: track 45.3 -> 43.3 mm
- net Col 1: track 74.8 -> 75.5 mm
Changed lines of the file:
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@@
 			(plot_on_all_layers_selection 0x00000000_00000000_00000000_00000000)
 			(disableapertmacros no)
-			(usegerberextensions no)
-			(usegerberattributes yes)
-			(usegerberadvancedattributes yes)
-			(creategerberjobfile yes)
+			(usegerberextensions yes)
+			(usegerberattributes no)
+			(usegerberadvancedattributes no)
+			(creategerberjobfile no)
 			(dashed_line_dash_ratio 12.000000)
 			(dashed_line_gap_ratio 3.000000)
@@
 			(sketchdnponfab yes)
 			(crossoutdnponfab yes)
-			(subtractmaskfromsilk no)
+			(subtractmaskfromsilk yes)
 			(outputformat 1)
 			(mirror no)
-			(drillshape 1)
+			(drillshape 0)
 			(scaleselection 1)
-			(outputdirectory "")
+			(outputdirectory "gerbers/")
 		)
 	)
@@
 			(at 7.62 -3.81 0)
 			(layer "F.SilkS")
+			(hide yes)
 			(effects
 				(font
@@
 		(start 190.373 105.918)
 		(end 190.373 113.284)
-		(width 0.16)
+		(width 0.3)
 		(layer "B.Cu")
 		(net 12)
@@
 		(start 189.738 106.807)
 		(end 189.738 114.173)
-		(width 0.16)
+		(width 0.3)
 		(layer "B.Cu")
 		(net 13)
@@
 	)
 	(segment
-		(start 193.802 120.142)
-		(end 195.326 120.142)
-		(width 0.3)
-		(layer "B.Cu")
-		(net 15)
-	)
-	(segment
 		(start 178.943 133.985)
 		(end 185.801 127.127)
@@
 	)
 	(segment
-		(start 192.913 121.031)
-		(end 193.802 120.142)
-		(width 0.3)
-		(layer "B.Cu")
-		(net 15)
-	)
-	(segment
 		(start 185.801 127.127)
 		(end 191.008 127.127)
@@
 	)
 	(segment
-		(start 165.481 133.985)
-		(end 178.943 133.985)
+		(start 193.675 120.269)
+		(end 196.088 120.269)
 		(width 0.3)
 		(layer "B.Cu")
@@
 	)
 	(segment
-		(start 164.973 100.838)
-		(end 164.973 116.84)
+		(start 192.913 121.031)
+		(end 193.675 120.269)
 		(width 0.3)
 		(layer "B.Cu")
@@
 	)
 	(segment
-		(start 164.465 119.38)
-		(end 164.465 132.969)
+		(start 165.481 133.985)
+		(end 178.943 133.985)
 		(width 0.3)
 		(layer "B.Cu")
@@
 	)
 	(segment
-		(start 195.199 88.9)
-		(end 196.088 89.789)
+		(start 164.973 100.838)
+		(end 164.973 116.84)
 		(width 0.3)
 		(layer "B.Cu")
-		(net 16)
-	)
-	(segment
-		(start 183.657 97.775)
-		(end 182.499 98.933)
-		(width 0.16)
-		(layer "B.Cu")
-		(net 16)
+		(net 15)
 	)
 	(segment
-		(start 182.499 99.314)
-		(end 183.642 98.171)
+		(start 164.465 119.38)
+		(end 164.465 132.969)
 		(width 0.3)
 		(layer "B.Cu")
-		(net 16)
+		(net 15)
 	)
 	(segment
-		(start 183.642 97.282)
-		(end 183.657 97.267)
+		(start 195.199 88.9)
+		(end 196.088 89.789)
 		(width 0.3)
 		(layer "B.Cu")
@@
 	)
 	(segment
-		(start 183.642 98.171)
-		(end 183.642 97.282)
+		(start 183.657 90.13)
+		(end 183.657 97.902)
 		(width 0.3)
 		(layer "B.Cu")
@@
 	)
 	(segment
-		(start 183.657 97.267)
-		(end 183.657 90.13)
+		(start 183.657 90.13)
+		(end 184.887 88.9)
 		(width 0.3)
 		(layer "B.Cu")
@@
 	)
 	(segment
-		(start 182.499 98.933)
-		(end 182.499 99.314)
-		(width 0.16)
-		(layer "B.Cu")
-		(net 16)
-	)
-	(segment
-		(start 183.657 90.13)
-		(end 184.887 88.9)
+		(start 183.657 97.902)
+		(end 182.499 99.06)
 		(width 0.3)
 		(layer "B.Cu")
@@
 		(width 0.3)
 		(layer "B.Cu")
+		(net 16)
+	)
+	(segment
+		(start 182.499 99.06)
+		(end 182.499 99.314)
+		(width 0.3)
+		(layer "B.Cu")
